File: STM32F030F4/Hardware/v5/STM32F030 - VGA minimal v5.brd (EAGLE design)
At the start: 25.4 x 17.8 mm, 28 parts, among them Q1 3904, U1 MCP1700/TT, U2 STM32F030F4P6, X1 25MHz

Commit message: Zener diodes value change
Parts:
- D1, D2: value 3V3 Zener -> 5V1 Zener
Changed lines of the file:
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@@
 <attribute name="VALUE" x="12.5785" y="2.9156" size="1.27" layer="27" font="vector" ratio="10" rot="R90"/>
 </element>
-<element name="D1" library="Misc Passives" package="SOD-123" value="3V3 Zener" x="19.05" y="12.573" smashed="yes" rot="MR270">
+<element name="D1" library="Misc Passives" package="SOD-123" value="5V1 Zener" x="19.05" y="12.573" smashed="yes" rot="MR270">
 <attribute name="NAME" x="17.9324" y="13.1572" size="0.4064" layer="26" rot="MR270"/>
-<attribute name="PARTNO" value="BZT52C3V3" x="19.05" y="12.573" size="1.778" layer="28" rot="MR270" display="off"/>
+<attribute name="PARTNO" value="BZT52C5V1" x="19.05" y="12.573" size="1.778" layer="28" rot="MR270" display="off"/>
 </element>
-<element name="D2" library="Misc Passives" package="SOD-123" value="3V3 Zener" x="21.59" y="12.573" smashed="yes" rot="MR270">
+<element name="D2" library="Misc Passives" package="SOD-123" value="5V1 Zener" x="21.59" y="12.573" smashed="yes" rot="MR270">
 <attribute name="NAME" x="22.3774" y="14.5796" size="0.4064" layer="26" rot="MR180"/>
-<attribute name="PARTNO" value="BZT52C3V3" x="21.59" y="12.573" size="1.778" layer="28" rot="MR270" display="off"/>
+<attribute name="PARTNO" value="BZT52C5V1" x="21.59" y="12.573" size="1.778" layer="28" rot="MR270" display="off"/>
 </element>
 <element name="J2" library="Misc Conn" package="1X04" value="" x="20.32" y="3.81" smashed="yes" rot="R180">
